Commit message: xarm poses

File: xarm_description/srdf/_xarm7_macro.srdf.xacro (robot description, xacro)
@@ -73,9 +73,9 @@
     <group_state name="home" group="${prefix}xarm7">
       <joint name="${prefix}joint1" value="0" />
-      <joint name="${prefix}joint2" value="0" />
+      <joint name="${prefix}joint2" value="-.7" />
       <joint name="${prefix}joint3" value="0" />
       <joint name="${prefix}joint4" value="0" />
       <joint name="${prefix}joint5" value="0" />
-      <joint name="${prefix}joint6" value="0" />
+      <joint name="${prefix}joint6" value=".7" />
       <joint name="${prefix}joint7" value="0" />
     </group_state>
@@ -88,4 +88,13 @@
       <joint name="${prefix}joint6" value="-1.5708" />
       <joint name="${prefix}joint7" value="0" />
+    </group_state>
+    <group_state name="vertical" group="xarm7">
+        <joint name="joint1" value="0.41" />
+        <joint name="joint2" value="-0.9786" />
+        <joint name="joint3" value="-0.1068" />
+        <joint name="joint4" value="0.7339" />
+        <joint name="joint5" value="-0.2118" />
+        <joint name="joint6" value="1.2559" />
+        <joint name="joint7" value="-0.4934" />
     </group_state>
     <!-- gripper -->

Commit message: recalibration of OUR borken arm

File: xarm_description/srdf/_xarm7_macro.srdf.xacro (robot description, xacro)
@@ -97,4 +97,13 @@
         <joint name="joint6" value="1.2559" />
         <joint name="joint7" value="-0.4934" />
+    </group_state>
+     <group_state name="close_up" group="xarm7">
+        <joint name="joint1" value="-1.4053" />
+        <joint name="joint2" value="-1.3522" />
+        <joint name="joint3" value="2.2036" />
+        <joint name="joint4" value="0.5622" />
+        <joint name="joint5" value="-0.5051" />
+        <joint name="joint6" value="-1.5978" />
+        <joint name="joint7" value="-0.8709" />
     </group_state>
     <!-- gripper -->

File: xarm_description/urdf/xarm7.urdf.xacro (robot description, xacro)
@@ -103,5 +103,5 @@
     <origin
       xyz="0 0 0.267"
-      rpy="0 0 0" />
+      rpy="0 0 -0.10472" />
     <parent
       link="${prefix}link_base" />
@@ -217,5 +217,5 @@
     <origin
       xyz="0 -0.293 0"
-      rpy="1.5708 0 0" />
+      rpy="1.5708 -.10472 0" />
     <parent
       link="${prefix}link2" />
@@ -331,5 +331,5 @@
     <origin
       xyz="0.0775 -0.3425 0"
-      rpy="1.5708 0 0" />
+      rpy="1.5708 .116937 0" />
     <parent
       link="${prefix}link4" />
@@ -445,5 +445,5 @@
     <origin
       xyz="0.076 0.097 0"
-      rpy="-1.5708 0 0" />
+      rpy="-1.5708 .174 0" />
     <parent
       link="${prefix}link6" />

File: xarm_gripper/urdf/xarm_gripper.urdf.xacro (robot description, xacro)
@@ -485,5 +485,5 @@
     type="fixed">
     <origin
-      xyz="0 0 0.1"
+      xyz="0 0 0.03"
       rpy="0 0  0" />
     <parent
